File: MainBoard/Kicad/FR4/ThreeDeeO.sch (KiCad schematic (older format))
At the start: 59 parts, among them J1 3-1775333-2, J10 S, J11 S, J12 B, J13 S, J2 JTAG, J3 S, J4 R, J5 G, J6 B, J8 S, J9 S, SW1 SW_DIP_x10, U1 ADV7125-lqfp48, U2 5M160ZE64I5N, U3 7WB383MUTAG, U4 7WB383MUTAG, U5 NVT2006BQ_115, U6 TPS73733DRVR, U7 MIC94310

Commit message: Minor updates
Parts:
- R21: value 330 -> 1K
- R5: value 523 -> 510
Changed lines of the file:
@@
 P 6050 1400
 F 0 "R5" V 5950 1350 50  0000 C CNN
-F 1 "523" V 5950 1450 50  0000 C CNN
+F 1 "510" V 5950 1550 50  0000 C CNN
 F 2 "Resistors_SMD:R_0402" H 6050 1400 50  0001 C CNN
 F 3 "~" H 6050 1400 50  0001 C CNN
@@
 P 5850 4200
 F 0 "R21" V 5750 4000 50  0000 C CNN
-F 1 "330" V 5850 4000 50  0000 C CNN
+F 1 "1K" V 5850 4000 50  0000 C CNN
 F 2 "Resistors_SMD:R_0402" H 5850 4200 50  0001 C CNN
 F 3 "~" H 5850 4200 50  0001 C CNN
